Commit message: バラ積み爪・THF を CAD から取り込み、PPO 学習を追加
- 爪 (pile-nail-v1) と Think Hand F の STL を tools/convert_meshes.py で URDF 用に変換。
  爪の当たり判定は長さ方向に切った凸包、先端 10mm は滑り止め (NITTO テープ) として別の凸包
- 左右の爪同士だけ当たり判定を有効化、グリッパの開きを全ストロークに、初期姿勢を開いた状態に
- 報酬をポテンシャル差分 (近くで粘っても貯まらない) に変更
- tools/train_ppo.py: スクリプト方策からの DAgger/DART で模倣してから PPO で微調整

Co-Authored-By: Claude Opus 5.5 <noreply@anthropic.com>

File: thinker-TMA-F1-REFX4-U3.urdf (robot description, URDF)
Before this commit: robot thinker-TMA-F1-REFX4-U3, 38 links, 37 joints
Links:
- link f1_thinker_TF1_nail_link: geometry collision mesh filename=package://thinker_ros2_description/nails/thinker-TF1/meshes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; collision mesh filename=package://thinker_ros2_description/nails/thinker-TF1/meshes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
- link f2_thinker_TF1_nail_link: geometry collision mesh filename=package://thinker_ros2_description/nails/thinker-TF1/meshes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; collision mesh filename=package://thinker_ros2_description/nails/thinker-TF1/meshes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
Joints:
- joint f1_thinker_TF1_tip_joint: origin xyz=0 0.0153 0.034 rpy=0 0 0.0 -> xyz=0 0.0238 0.045 rpy=0 0 0.0
- joint f2_thinker_TF1_tip_joint: origin xyz=0 0.0153 0.034 rpy=0 0 -3.141592653589793 -> xyz=0 0.0238 0.045 rpy=0 0 -3.141592653589793

Commit message: Hand-E と THF のアダプタを CAD から取り込み、THF をアダプタに合わせて配置、f1/f2 を left/right に改名
- packages/thf-hande-adapter-v3.stl を tools/convert_meshes.py で Hand-E の指フレームに変換して左右の指スライダーに付けた。
  座ぐり穴 (間隔 9mm) が Hand-E の指取付ねじ穴 (robotiq_hande_description の finger.dae) に、
  溝が指スライダーの凸部 (幅 6, 高さ 1mm) に合う向き
- THF のタブ (M3 穴 2 個、間隔 14mm) がアダプタのポケットに入る位置に base_joint を変更。
  THF は外へ (左は +x、右は -x 側から見て内へ) 3.9mm、上へ 4.7mm ずれ、全閉の爪先が -11.2 / +3.4mm の偏りから ±7.3mm の左右対称になった
- 仮の指スライダーの箱を、Hand-E の上面から出ている凸部の寸法に変更
- THF のリンク・関節名と爪の状態のキーを f1/f2 から left/right に (f1 が左指)。観測の並びは同じなので既存のチェックポイントはそのまま読める

Co-Authored-By: Claude Opus 5.5 <noreply@anthropic.com>

File: thinker-TMA-F1-REFX4-U3.urdf (robot description, URDF)
Before this commit: robot thinker-TMA-F1-REFX4-U3, 38 links, 37 joints
Links:
- removed link f1_thinker_TF1_base_link
- removed link f1_thinker_TF1_nail_link
- removed link f1_thinker_TF1_nail_mount_link
- removed link f1_thinker_TF1_tip_link
- removed link f1_thinker_TF1_x_link
- removed link f1_thinker_TF1_y_link
- removed link f1_thinker_TF1_z_link
- removed link f2_thinker_TF1_base_link
- removed link f2_thinker_TF1_nail_link
- removed link f2_thinker_TF1_nail_mount_link
- removed link f2_thinker_TF1_tip_link
- removed link f2_thinker_TF1_x_link
- removed link f2_thinker_TF1_y_link
- removed link f2_thinker_TF1_z_link
- added link left_thinker_TF1_base_link, mass 0.285; collision mesh filename=package://thinker_ros2_description/fingers/thinker-TF1/mesh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; visual mesh filename=package://thinker_ros2_description/fingers/thinker-TF1/mesh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
- added link left_thinker_TF1_nail_link, mass 0.01; collision mesh filename=package://thinker_ros2_description/nails/thinker-TF1/meshes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; collision mesh filename=package://thinker_ros2_description/nails/thinker-TF1/meshes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
- added link left_thinker_TF1_nail_mount_link, mass 0.001; visual box size=0.001 0.001 0.001
- added link left_thinker_TF1_tip_link, mass 0.001; visual box size=0.001 0.001 0.001
- added link left_thinker_TF1_x_link, mass 0.01; visual mesh filename=package://thinker_ros2_description/fingers/thinker-TF1/mesh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
- added link left_thinker_TF1_y_link, mass 0.01; visual mesh filename=package://thinker_ros2_description/fingers/thinker-TF1/mesh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
- added link left_thinker_TF1_z_link, mass 0.03; visual mesh filename=package://thinker_ros2_description/fingers/thinker-TF1/mesh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
- added link right_thinker_TF1_base_link, mass 0.285; collision mesh filename=package://thinker_ros2_description/fingers/thinker-TF1/mesh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; visual mesh filename=package://thinker_ros2_description/fingers/thinker-TF1/mesh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
- added link right_thinker_TF1_nail_link, mass 0.01; collision mesh filename=package://thinker_ros2_description/nails/thinker-TF1/meshes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; collision mesh filename=package://thinker_ros2_description/nails/thinker-TF1/meshes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
- added link right_thinker_TF1_nail_mount_link, mass 0.001; visual box size=0.001 0.001 0.001
- added link right_thinker_TF1_tip_link, mass 0.001; visual box size=0.001 0.001 0.001
- added link right_thinker_TF1_x_link, mass 0.01; visual mesh filename=package://thinker_ros2_description/fingers/thinker-TF1/mesh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
- added link right_thinker_TF1_y_link, mass 0.01; visual mesh filename=package://thinker_ros2_description/fingers/thinker-TF1/mesh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
- added link right_thinker_TF1_z_link, mass 0.03; visual mesh filename=package://thinker_ros2_description/fingers/thinker-TF1/mesh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
- link robotiq_hande_left_finger: geometry collision mesh filename=package://thinker_ros2_description/fingers/thinker-TF1/mesh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; visual mesh filename=package://thinker_ros2_description/fingers/thinker-TF1/mesh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
- link robotiq_hande_right_finger: geometry collision mesh filename=package://thinker_ros2_description/fingers/thinker-TF1/mesh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; visual mesh filename=package://thinker_ros2_description/fingers/thinker-TF1/mesh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
Joints:
- removed joint f1_thinker_TF1_base_joint
- removed joint f1_thinker_TF1_nail_joint
- removed joint f1_thinker_TF1_nail_mount_joint
- removed joint f1_thinker_TF1_tip_joint
- removed joint f1_thinker_TF1_x_joint
- removed joint f1_thinker_TF1_y_joint
- removed joint f1_thinker_TF1_z_joint
- removed joint f2_thinker_TF1_base_joint
- removed joint f2_thinker_TF1_nail_joint
- removed joint f2_thinker_TF1_nail_mount_joint
- removed joint f2_thinker_TF1_tip_joint
- removed joint f2_thinker_TF1_x_joint
- removed joint f2_thinker_TF1_y_joint
- removed joint f2_thinker_TF1_z_joint
- added joint left_thinker_TF1_base_joint: type fixed, parent robotiq_hande_left_finger, child left_thinker_TF1_base_link, origin xyz=0.0219 0 0.0058 rpy=0 0 3.141592653589793
- added joint left_thinker_TF1_nail_joint: type fixed, parent left_thinker_TF1_nail_mount_link, child left_thinker_TF1_nail_link, origin xyz=0 0.0015 0 rpy=0 0 0
- added joint left_thinker_TF1_nail_mount_joint: type fixed, parent left_thinker_TF1_z_link, child left_thinker_TF1_nail_mount_link, origin xyz=0 0 0.0276 rpy=0 0 0
- added joint left_thinker_TF1_tip_joint: type fixed, parent left_thinker_TF1_nail_link, child left_thinker_TF1_tip_link, origin xyz=0 0.0238 0.045 rpy=0 0 0.0
- added joint left_thinker_TF1_x_joint: type revolute, parent left_thinker_TF1_base_link, child left_thinker_TF1_x_link, origin xyz=0 0 0.0373 rpy=-1.5707963267948966 0 0, axis 0 0 1, limit lower=-0.12217304763960307 upper=0.12217304763960307 effort=20.0 velocity=2.00
- added joint left_thinker_TF1_y_joint: type revolute, parent left_thinker_TF1_x_link, child left_thinker_TF1_y_link, origin xyz=0 0 0 rpy=0 1.5707963267948966 0, axis 0 0 1, limit lower=-0.12217304763960307 upper=0.12217304763960307 effort=20.0 velocity=6.28
- added joint left_thinker_TF1_z_joint: type prismatic, parent left_thinker_TF1_y_link, child left_thinker_TF1_z_link, origin xyz=0 0 0.0039 rpy=1.5707963267948966 0 0, axis 0 0 -1, limit lower=0.0 upper=0.0039 effort=1000.0 velocity=10.0
- added joint right_thinker_TF1_base_joint: type fixed, parent robotiq_hande_right_finger, child right_thinker_TF1_base_link, origin xyz=-0.0141 0 0.0058 rpy=0 0 3.141592653589793
- added joint right_thinker_TF1_nail_joint: type fixed, parent right_thinker_TF1_nail_mount_link, child right_thinker_TF1_nail_link, origin xyz=0 -0.0015 0 rpy=0 0 3.141592653589793
- added joint right_thinker_TF1_nail_mount_joint: type fixed, parent right_thinker_TF1_z_link, child right_thinker_TF1_nail_mount_link, origin xyz=0 0 0.0276 rpy=0 0 0
- added joint right_thinker_TF1_tip_joint: type fixed, parent right_thinker_TF1_nail_link, child right_thinker_TF1_tip_link, origin xyz=0 0.0238 0.045 rpy=0 0 -3.141592653589793
- added joint right_thinker_TF1_x_joint: type revolute, parent right_thinker_TF1_base_link, child right_thinker_TF1_x_link, origin xyz=0 0 0.0373 rpy=-1.5707963267948966 0 0, axis 0 0 1, limit lower=-0.12217304763960307 upper=0.12217304763960307 effort=20.0 velocity=2.00
- added joint right_thinker_TF1_y_joint: type revolute, parent right_thinker_TF1_x_link, child right_thinker_TF1_y_link, origin xyz=0 0 0 rpy=0 1.5707963267948966 0, axis 0 0 1, limit lower=-0.12217304763960307 upper=0.12217304763960307 effort=20.0 velocity=6.28
- added joint right_thinker_TF1_z_joint: type prismatic, parent right_thinker_TF1_y_link, child right_thinker_TF1_z_link, origin xyz=0 0 0.0039 rpy=1.5707963267948966 0 0, axis 0 0 -1, limit lower=0.0 upper=0.0039 effort=1000.0 velocity=10.0
