Commit message: newton physicsで動作テスト

File: thinker-TMA-F1-REFX4-U3.urdf (robot description, URDF)
Before this commit: robot thinker-TMA-F1-REFX4-U3, 38 links, 37 joints
Joints:
- joint f1_thinker_TF1_x_joint: limit lower=-0.17453292519943295 upper=0.17453292519943295 effort=20.0 velocity=2.00 -> lower=-0.12217304763960307 upper=0.12217304763960307 effort=20.0 velocity=2.00
- joint f1_thinker_TF1_y_joint: limit lower=-0.17453292519943295 upper=0.17453292519943295 effort=20.0 velocity=6.28 -> lower=-0.12217304763960307 upper=0.12217304763960307 effort=20.0 velocity=6.28
- joint f1_thinker_TF1_z_joint: limit lower=0.0 upper=0.005 effort=1000.0 velocity=10.0 -> lower=0.0 upper=0.004 effort=1000.0 velocity=10.0
- joint f2_thinker_TF1_x_joint: limit lower=-0.17453292519943295 upper=0.17453292519943295 effort=20.0 velocity=2.00 -> lower=-0.12217304763960307 upper=0.12217304763960307 effort=20.0 velocity=2.00
- joint f2_thinker_TF1_y_joint: limit lower=-0.17453292519943295 upper=0.17453292519943295 effort=20.0 velocity=6.28 -> lower=-0.12217304763960307 upper=0.12217304763960307 effort=20.0 velocity=6.28
- joint f2_thinker_TF1_z_joint: limit lower=0.0 upper=0.005 effort=1000.0 velocity=10.0 -> lower=0.0 upper=0.004 effort=1000.0 velocity=10.0

Commit message: THF爪可動範囲を±10degから±7degに、zは0を無接触状態、-3.9を最大押し込み状態とした

File: thinker-TMA-F1-REFX4-U3.urdf (robot description, URDF)
Before this commit: robot thinker-TMA-F1-REFX4-U3, 38 links, 37 joints
Joints:
- joint f1_thinker_TF1_z_joint: limit lower=0.0 upper=0.004 effort=1000.0 velocity=10.0 -> lower=-0.0039 upper=0.0 effort=1000.0 velocity=10.0; origin xyz=0 0 0 rpy=1.5707963267948966 0 0 -> xyz=0 0 0.0039 rpy=1.5707963267948966 0 0
- joint f2_thinker_TF1_z_joint: limit lower=0.0 upper=0.004 effort=1000.0 velocity=10.0 -> lower=-0.0039 upper=0.0 effort=1000.0 velocity=10.0; origin xyz=0 0 0 rpy=1.5707963267948966 0 0 -> xyz=0 0 0.0039 rpy=1.5707963267948966 0 0

Commit message: tma, newtonでの把持テスト

File: thinker-TMA-F1-REFX4-U3.urdf (robot description, URDF)
Before this commit: robot thinker-TMA-F1-REFX4-U3, 38 links, 37 joints
Joints:
- joint f1_thinker_TF1_z_joint: axis 0 0 1 -> 0 0 -1; limit lower=-0.0039 upper=0.0 effort=1000.0 velocity=10.0 -> lower=0.0 upper=0.0039 effort=1000.0 velocity=10.0
- joint f2_thinker_TF1_z_joint: axis 0 0 1 -> 0 0 -1; limit lower=-0.0039 upper=0.0 effort=1000.0 velocity=10.0 -> lower=0.0 upper=0.0039 effort=1000.0 velocity=10.0

Commit message: thfの構造修正

File: thinker-TMA-F1-REFX4-U3.urdf (robot description, URDF)
Before this commit: robot thinker-TMA-F1-REFX4-U3, 38 links, 37 joints
Joints:
- joint left_thinker_TF1_nail_joint: origin xyz=0 0.0015 0 rpy=0 0 0 -> xyz=0 0.0003 0 rpy=0 0 0
- joint right_thinker_TF1_nail_joint: origin xyz=0 -0.0015 0 rpy=0 0 3.141592653589793 -> xyz=0 -0.0003 0 rpy=0 0 3.141592653589793
