Commit message: ファイル整理

File: tma.urdf (robot description, URDF)
Before this commit: robot thinker-TMA-F1-REFX4-U3, 38 links, 37 joints
Links:
- removed link left_thinker_TF1_base_link
- removed link left_thinker_TF1_nail_link
- removed link left_thinker_TF1_nail_mount_link
- removed link left_thinker_TF1_tip_link
- removed link left_thinker_TF1_x_link
- removed link left_thinker_TF1_y_link
- removed link left_thinker_TF1_z_link
- removed link right_thinker_TF1_base_link
- removed link right_thinker_TF1_nail_link
- removed link right_thinker_TF1_nail_mount_link
- removed link right_thinker_TF1_tip_link
- removed link right_thinker_TF1_x_link
- removed link right_thinker_TF1_y_link
- removed link right_thinker_TF1_z_link
- added link left_thf_base_link, mass 0.285; collision mesh filename=package://think_hand_f_description/fingers/thinker-TF1/mesh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; visual mesh filename=package://think_hand_f_description/fingers/thinker-TF1/mesh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
- added link left_thf_nail_link, mass 0.01; collision mesh filename=package://think_hand_f_description/nails/thinker-TF1/meshes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; collision mesh filename=package://think_hand_f_description/nails/thinker-TF1/meshes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
- added link left_thf_nail_mount_link, mass 0.001; visual box size=0.001 0.001 0.001
- added link left_thf_tip_link, mass 0.001; visual box size=0.001 0.001 0.001
- added link left_thf_x_link, mass 0.01; visual mesh filename=package://think_hand_f_description/fingers/thinker-TF1/mesh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
- added link left_thf_y_link, mass 0.01; visual mesh filename=package://think_hand_f_description/fingers/thinker-TF1/mesh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
- added link left_thf_z_link, mass 0.03; visual mesh filename=package://think_hand_f_description/fingers/thinker-TF1/mesh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
- added link right_thf_base_link, mass 0.285; collision mesh filename=package://think_hand_f_description/fingers/thinker-TF1/mesh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; visual mesh filename=package://think_hand_f_description/fingers/thinker-TF1/mesh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
- added link right_thf_nail_link, mass 0.01; collision mesh filename=package://think_hand_f_description/nails/thinker-TF1/meshes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; collision mesh filename=package://think_hand_f_description/nails/thinker-TF1/meshes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
- added link right_thf_nail_mount_link, mass 0.001; visual box size=0.001 0.001 0.001
- added link right_thf_tip_link, mass 0.001; visual box size=0.001 0.001 0.001
- added link right_thf_x_link, mass 0.01; visual mesh filename=package://think_hand_f_description/fingers/thinker-TF1/mesh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
- added link right_thf_y_link, mass 0.01; visual mesh filename=package://think_hand_f_description/fingers/thinker-TF1/mesh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
- added link right_thf_z_link, mass 0.03; visual mesh filename=package://think_hand_f_description/fingers/thinker-TF1/mesh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
- link robotiq_hande_left_finger: geometry collision mesh filename=package://think_hand_f_description/fingers/thinker-TF1/mesh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; visual mesh filename=package://think_hand_f_description/fingers/thinker-TF1/mesh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
- link robotiq_hande_right_finger: geometry collision mesh filename=package://think_hand_f_description/fingers/thinker-TF1/mesh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; visual mesh filename=package://think_hand_f_description/fingers/thinker-TF1/mesh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
- link thinker_camera_link: geometry collision box size=0.023 0.042 0.042; visual mesh filename=package://realsense2_description/meshes/d405-body.stl scale=0.001 0.001 0.001
Joints:
- removed joint left_thinker_TF1_base_joint
- removed joint left_thinker_TF1_nail_joint
- removed joint left_thinker_TF1_nail_mount_joint
- removed joint left_thinker_TF1_tip_joint
- removed joint left_thinker_TF1_x_joint
- removed joint left_thinker_TF1_y_joint
- removed joint left_thinker_TF1_z_joint
- removed joint right_thinker_TF1_base_joint
- removed joint right_thinker_TF1_nail_joint
- removed joint right_thinker_TF1_nail_mount_joint
- removed joint right_thinker_TF1_tip_joint
- removed joint right_thinker_TF1_x_joint
- removed joint right_thinker_TF1_y_joint
- removed joint right_thinker_TF1_z_joint
- added joint left_thf_base_joint: type fixed, parent robotiq_hande_left_finger, child left_thf_base_link, origin xyz=0.0219 0 0.0058 rpy=0 0 3.141592653589793
- added joint left_thf_nail_joint: type fixed, parent left_thf_nail_mount_link, child left_thf_nail_link, origin xyz=0 0.0003 0 rpy=0 0 0
- added joint left_thf_nail_mount_joint: type fixed, parent left_thf_z_link, child left_thf_nail_mount_link, origin xyz=0 0 0.0276 rpy=0 0 0
- added joint left_thf_tip_joint: type fixed, parent left_thf_nail_link, child left_thf_tip_link, origin xyz=0 0.0238 0.045 rpy=0 0 0.0
- added joint left_thf_x_joint: type revolute, parent left_thf_base_link, child left_thf_x_link, origin xyz=0 0 0.0373 rpy=-1.5707963267948966 0 0, axis 0 0 1, limit lower=-0.12217304763960307 upper=0.12217304763960307 effort=20.0 velocity=2.00
- added joint left_thf_y_joint: type revolute, parent left_thf_x_link, child left_thf_y_link, origin xyz=0 0 0 rpy=0 1.5707963267948966 0, axis 0 0 1, limit lower=-0.12217304763960307 upper=0.12217304763960307 effort=20.0 velocity=6.28
- added joint left_thf_z_joint: type prismatic, parent left_thf_y_link, child left_thf_z_link, origin xyz=0 0 0.0039 rpy=1.5707963267948966 0 0, axis 0 0 -1, limit lower=0.0 upper=0.0039 effort=1000.0 velocity=10.0
- added joint right_thf_base_joint: type fixed, parent robotiq_hande_right_finger, child right_thf_base_link, origin xyz=-0.0141 0 0.0058 rpy=0 0 3.141592653589793
- added joint right_thf_nail_joint: type fixed, parent right_thf_nail_mount_link, child right_thf_nail_link, origin xyz=0 -0.0003 0 rpy=0 0 3.141592653589793
- added joint right_thf_nail_mount_joint: type fixed, parent right_thf_z_link, child right_thf_nail_mount_link, origin xyz=0 0 0.0276 rpy=0 0 0
- added joint right_thf_tip_joint: type fixed, parent right_thf_nail_link, child right_thf_tip_link, origin xyz=0 0.0238 0.045 rpy=0 0 -3.141592653589793
- added joint right_thf_x_joint: type revolute, parent right_thf_base_link, child right_thf_x_link, origin xyz=0 0 0.0373 rpy=-1.5707963267948966 0 0, axis 0 0 1, limit lower=-0.12217304763960307 upper=0.12217304763960307 effort=20.0 velocity=2.00
- added joint right_thf_y_joint: type revolute, parent right_thf_x_link, child right_thf_y_link, origin xyz=0 0 0 rpy=0 1.5707963267948966 0, axis 0 0 1, limit lower=-0.12217304763960307 upper=0.12217304763960307 effort=20.0 velocity=6.28
- added joint right_thf_z_joint: type prismatic, parent right_thf_y_link, child right_thf_z_link, origin xyz=0 0 0.0039 rpy=1.5707963267948966 0 0, axis 0 0 -1, limit lower=0.0 upper=0.0039 effort=1000.0 velocity=10.0
