Commit message: THF の質量を製品仕様 (本体 250g、グリッパ部を除く) に合わせる
片側 125g から可動部 (62g) を引いた 63g を base_link に入れ、重心・慣性は当たり判定の凸包から計算した。
以前の値 (285g、重心が外形の外) は片側 347g、左右で約 700g になっていた。cobotta.urdf も再生成。

Co-Authored-By: Claude Opus 5.5 <noreply@anthropic.com>

File: cobotta.urdf (robot description, URDF)
Before this commit: robot thinker_cobotta, 25 links, 24 joints
Links:
- link left_thf_base_link: mass 0.285 -> 0.063
- link right_thf_base_link: mass 0.285 -> 0.063

File: tma.urdf (robot description, URDF)
Before this commit: robot thinker-model-a, 38 links, 37 joints
Links:
- link left_thf_base_link: mass 0.285 -> 0.063
- link right_thf_base_link: mass 0.285 -> 0.063
